File: frustratedfly.kicad_sch (KiCad schematic)
At the start: 73 parts, among them SW1 CPG1316S, SW10 CPG1316S, SW11 CPG1316S, SW12 CPG1316S, SW13 CPG1316S, SW14 CPG1316S, SW15 CPG1316S, SW16 CPG1316S, SW17 CPG1316S, SW18 CPG1316S, SW19 CPG1316S, SW2 CPG1316S, SW20 CPG1316S, SW21 CPG1316S, SW22 CPG1316S, SW23 CPG1316S, SW24 CPG1316S, SW25 CPG1316S, SW26 CPG1316S, SW27 CPG1316S, SW28 CPG1316S, SW29 CPG1316S, SW3 CPG1316S, SW30 CPG1316S, SW31 CPG1316S, SW32 CPG1316S, SW33 CPG1316S, SW34 CPG1316S, SW35 CPG1316S, SW36 CPG1316S, SW4 CPG1316S, SW5 CPG1316S, SW6 CPG1316S, SW7 CPG1316S, SW8 CPG1316S, SW9 CPG1316S

Commit message: Added project specific kicad libs
Parts:
- RZ1: footprint Keyboard_stuff:RP2040_Zero_cutout -> frustratedfly:RP2040_Zero_cutout; symbol Keyboard_stuff:RP2040-Zero -> frustratedfly:RP2040-Zero; now in the parts list
- SW1, SW10, SW11, SW12, SW13, SW14, SW15, SW16, SW17, SW18, SW19, SW2, SW20, SW21, SW22, SW23, SW24, SW25, SW26, SW27, SW28, SW29, SW3, SW30, SW31, SW32, SW33, SW34, SW35, SW36, SW4, SW5, SW6, SW7, SW8, SW9: footprint Keyboard_stuff:CPG1316S01D02_mikeholscher_w_ref -> frustratedfly:CPG1316S01D02_mikeholscher_w_ref
